File: motor controller.kicad_pcb (KiCad board)
At the start: 2 copper layers, 55 parts, among them J1 Servo Header, J2 XT30, J3 Ext Power, J4 USB_PWR, J5 USB Header, J6 M0, J7 M1, J8 M2, J9 M3, M0-BUF1 SN74LVC2G14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

Commit message: updated schematic and pcb
Parts:
- removed IFX9201SG1: M1, 9201SG:PG_DSO_12_17
- removed IFX9201SG2: M3, 9201SG:PG_DSO_12_17
- removed IFX9201SG3: M2, 9201SG:PG_DSO_12_17
- removed IFX9201SG4: M0, 9201SG:PG_DSO_12_17
- added U1: M1-IFX9201SG, 9201SG:PG_DSO_12_17, F.Cu at (134.6, 79.2)
- added U2: M3-IFX9201SG, 9201SG:PG_DSO_12_17, F.Cu at (116.9, 75.7)
- added U3: M2-IFX9201SG, 9201SG:PG_DSO_12_17, F.Cu at (191.5, 77.2)
- added U4: M0-IFX9201SG, 9201SG:PG_DSO_12_17, F.Cu at (178.3, 80.3)
- J3: footprint Connector_AMASS:AMASS_XT30PW-M_1x02_P2.50mm_Horizontal -> Connector_JST:JST_XH_S3B-XH-A_1x03_P2.50mm_Horizontal
- M0DA1: footprint LED_SMD:LED_0805_2012Metric_Pad1.15x1.40mm_HandSolder -> LED_SMD:LED_0805_2012Metric
- SW1: value SW_Push -> RESET
- moved M2-BUF1 143.9 mm to (196.2, 64.9), turned to -90 degrees
- moved C20 139.8 mm to (112.8, 64.9), turned to 90 degrees
- moved C19 136.1 mm to (115.3, 64.9), turned to -90 degrees
- moved J8 133.0 mm to (196.4, 59.8), turned to 180 degrees
- moved M0-BUF1 126.4 mm to (185.4, 87.7), turned to 90 degrees
- moved C15 118.9 mm to (122.3, 87.4), turned to 90 degrees
- moved C16 117.5 mm to (124.9, 87.4), turned to -90 degrees
- moved C6 112.0 mm to (125.5, 79.8), turned to 90 degrees
- moved C4 111.3 mm to (129.5, 65.0), turned to 180 degrees
- moved J5 109.1 mm to (177.4, 59.8)
- moved C1 100.8 mm to (178.3, 70.1), turned to 0 degrees
- moved M3DB1 99.7 mm to (117.9, 64.4), turned to -90 degrees
- moved C3 98.4 mm to (139.7, 70.6), turned to 90 degrees
- moved C5 97.5 mm to (137.7, 85.3)
- moved M3DA1 96.8 mm to (119.9, 64.4), turned to -90 degrees
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Connections:
- C19 pad 2: M3-B -> M3-A
- C20 pad 1: M3-A -> M3-B
- M0-BUF1 pad 1: M0-Enc-A -> M0-Enc-B
- M0-BUF1 pad 3: M0-Enc-B -> M0-Enc-A
- M1-BUF1 pad 1: M1-Enc-A -> M1-Enc-B
- M1-BUF1 pad 3: M1-Enc-B -> M1-Enc-A
- M2-BUF1 pad 1: M2-Enc-A -> M2-Enc-B
- M2-BUF1 pad 3: M2-Enc-B -> M2-Enc-A
- M3-BUF1 pad 1: M3-Enc-A -> M3-Enc-B
- M3-BUF1 pad 3: M3-Enc-B -> M3-Enc-A
Routing:
- net 5v: track 0.00 -> 80.3 mm, vias 0 -> 1
- net +VM: track 0.00 -> 55.1 mm, vias 0 -> 9
- net GND: track 0.00 -> 26.3 mm
- net M1-A: track 0.00 -> 19.6 mm, vias 0 -> 2
- net Net-(A1-VBUS): track 0.00 -> 19.1 mm
- net M1-PWM: track 0.00 -> 18.1 mm
- net M1-B: track 0.00 -> 12.2 mm, vias 0 -> 2
- net M3-A: track 0.00 -> 11.1 mm
- net GPIO15: track 0.00 -> 9.65 mm
- net Net-(J4-Pin_1): track 0.00 -> 7.48 mm
- net M3-B: track 0.00 -> 7.14 mm
- net GPIO17: track 0.00 -> 7.03 mm
- net GPIO21: track 0.00 -> 6.80 mm
- net GPIO16: track 0.00 -> 6.63 mm
- net GPIO22: track 0.00 -> 6.56 mm
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Other:
- board outline added: 90.9 x 52.5 mm
- board text added: "EXT USB"

Commit message: fixed a short, started updating the PCB layout
Parts:
- removed C1, C10, C9: 100uF, Capacitor_THT:CP_Radial_D6.3mm_P2.50mm
- removed C17, C18, C19, C20: 10n, Capacitor_SMD:C_1206_3216Metric
- added C13: 22n, Capacitor_SMD:C_1206_3216Metric, F.Cu at (210.5, 85.5)
- added C14: 22n, Capacitor_SMD:C_1206_3216Metric, F.Cu at (210.5, 88.8)
- added C15: 22n, Capacitor_SMD:C_1206_3216Metric, F.Cu at (210.5, 92.2)
- added C16: 22n, Capacitor_SMD:C_1206_3216Metric, F.Cu at (210.5, 95.5)
- added C5: 22n, Capacitor_SMD:C_1206_3216Metric, F.Cu at (210.5, 72.0)
- added C6: 22n, Capacitor_SMD:C_1206_3216Metric, F.Cu at (210.5, 75.4)
- added C7: 22n, Capacitor_SMD:C_1206_3216Metric, F.Cu at (210.5, 78.8)
- added C8: 22n, Capacitor_SMD:C_1206_3216Metric, F.Cu at (210.5, 82.1)
- C11, C12, C13, C14, C3, C4, C5, C6: value 100n -> 22n
- C15, C16, C7, C8: value 10n -> 22n
- moved C2 43.6 mm to (216.2, 74.3), turned to 0 degrees
- renumbered M3-BUF1 to U5, M0-BUF1 to U6, M2-BUF1 to U7, M1-BUF1 to U8
Connections:
- net +VM renamed Vdrive
- net 12v renamed +12V
- A1 pad 36: 3.3v -> +3V3
- C13 pad 1: 3.3v -> GND
- C13 pad 2: Net-(U4-VSO) -> +3V3
- C14 pad 1: 3.3v -> GND
- C14 pad 2: Net-(U3-VSO) -> +3V3
- C15 pad 1: Net-(J7-Pin_5) -> GND
- C15 pad 2: M1-B -> +3V3
- C16 pad 1: M1-A -> GND
- C16 pad 2: Net-(J7-Pin_6) -> +3V3
- C5 pad 1: 3.3v -> +3V3
- C5 pad 2: Net-(U1-VSO) -> GND
- C6 pad 1: 3.3v -> +3V3
- C6 pad 2: Net-(U2-VSO) -> GND
- C7 pad 1: Net-(J6-Pin_5) -> +3V3
- C7 pad 2: M0-B -> GND
- C8 pad 1: M0-A -> +3V3
- C8 pad 2: Net-(J6-Pin_6) -> GND
- J3 pad 2: 5v -> +5V
- J6 pad 5: Net-(J6-Pin_5) -> M0-B
- J6 pad 6: Net-(J6-Pin_6) -> M0-A
- J7 pad 5: Net-(J7-Pin_5) -> M1-B
- J7 pad 6: Net-(J7-Pin_6) -> M1-A
- J8 pad 5: Net-(J8-Pin_5) -> M2-B
- J8 pad 6: Net-(J8-Pin_6) -> M2-A
- J9 pad 5: Net-(J9-Pin_5) -> M3-A
- J9 pad 6: Net-(J9-Pin_6) -> M3-B
- U1 pad 2: Net-(U1-VSO) -> +3V3
- U2 pad 2: Net-(U2-VSO) -> +3V3
- U3 pad 2: Net-(U3-VSO) -> +3V3
- U4 pad 2: Net-(U4-VSO) -> +3V3
- U5 pad 5: 5v -> +3V3
- U6 pad 5: 5v -> +3V3
- U7 pad 5: 5v -> +3V3
- U8 pad 5: 5v -> +3V3
Routing:
- net (no net): track 0.00 -> 16.4 mm
- net Net-(J8-Pin_5): track 4.29 -> 0.00 mm
- net M2-B: track 0.00 -> 4.29 mm
- net Net-(J8-Pin_6): track 4.27 -> 0.00 mm
- net M2-A: track 0.00 -> 4.27 mm
- net Net-(J7-Pin_6): track 4.11 -> 0.00 mm
- net Net-(J7-Pin_5): track 4.10 -> 0.00 mm
- net Net-(J6-Pin_6): track 4.09 -> 0.00 mm
- net Net-(J6-Pin_5): track 4.08 -> 0.00 mm
- net Net-(J9-Pin_5): track 3.89 -> 0.00 mm
- net M3-A: track 11.1 -> 15.0 mm
- net Net-(J9-Pin_6): track 3.87 -> 0.00 mm
- net M3-B: track 7.14 -> 11.0 mm

Commit message: more tweaking
Parts:
- removed the C13 at (210.5, 85.5)
- removed C14 (x2), C15 (x2), C16 (x2): 22n, Capacitor_SMD:C_1206_3216Metric
- removed the C5 at (210.5, 72.0)
- removed the C6 at (210.5, 75.4)
- removed the C7 at (210.5, 78.8)
- removed the C8 at (197.1, 87.3)
- removed the C8 at (210.5, 82.1)
- added C1: 22n, Capacitor_SMD:C_1206_3216Metric, F.Cu at (110.5, 87.7)
- added C10: 22n, Capacitor_SMD:C_1206_3216Metric, F.Cu at (120.2, 72.2)
- added C8: 22n, Capacitor_SMD:C_1206_3216Metric, F.Cu at (119.9, 80.2)
- added C9: 100uF, Capacitor_THT:CP_Radial_D6.3mm_P2.50mm, F.Cu at (175.2, 83.0)
- C2: value 100uF -> 22n; footprint Capacitor_THT:CP_Radial_D6.3mm_P2.50mm -> Capacitor_SMD:C_1206_3216Metric
- J2: value XT30 -> Ext Power; footprint Connector_AMASS:AMASS_XT30PW-M_1x02_P2.50mm_Horizontal -> Connector_JST:JST_XH_S3B-XH-A_1x03_P2.50mm_Horizontal
- J3: value Ext Power -> USB_PWR; footprint Connector_JST:JST_XH_S3B-XH-A_1x03_P2.50mm_Horizontal -> Connector_PinHeader_2.54mm:PinHeader_1x03_P2.54mm_Vertical
- J4: value USB_PWR -> USB Header; footprint Connector_PinHeader_2.54mm:PinHeader_1x03_P2.54mm_Vertical -> Connector_JST:JST_XH_S4B-XH-A_1x04_P2.50mm_Horizontal
- J5: value USB Header -> XT30; footprint Connector_JST:JST_XH_S4B-XH-A_1x04_P2.50mm_Horizontal -> Connector_AMASS:AMASS_XT30PW-M_1x02_P2.50mm_Horizontal
- U1: value M1-IFX9201SG -> SN74LVC2G14; footprint 9201SG:PG_DSO_12_17 -> Package_TO_SOT_SMD:SOT-23-6
- U2: value M3-IFX9201SG -> SN74LVC2G14; footprint 9201SG:PG_DSO_12_17 -> Package_TO_SOT_SMD:SOT-23-6
- U3: value M2-IFX9201SG -> M3-IFX9201SG
- U4: value M0-IFX9201SG -> M1-IFX9201SG
- U7: value SN74LVC2G14 -> M2-IFX9201SG; footprint Package_TO_SOT_SMD:SOT-23-6 -> 9201SG:PG_DSO_12_17
- U8: value SN74LVC2G14 -> M0-IFX9201SG; footprint Package_TO_SOT_SMD:SOT-23-6 -> 9201SG:PG_DSO_12_17
- moved C3 81.5 mm to (219.9, 85.2), turned to 180 degrees
- moved U8 78.7 mm to (190.6, 102.8), turned to 0 degrees
- moved U2 78.5 mm to (194.8, 65.4), turned to -90 degrees
- moved U3 75.7 mm to (116.5, 66.8), turned to 180 degrees
- moved U6 65.2 mm to (124.5, 64.6), turned to -90 degrees
- moved U4 64.1 mm to (118.3, 102.9)
- moved C12 56.7 mm to (124.7, 80.2)
- moved J3 51.0 mm to (174.5, 66.2), turned to -90 degrees
- moved U1 49.0 mm to (178.8, 100.3)
- moved J5 46.5 mm to (171.5, 106.0)
- moved J2 45.2 mm to (130.7, 110.0), turned to 0 degrees
- moved C5 44.9 mm to (179.8, 69.5), turned to 90 degrees
- moved C13 44.7 mm to (215.2, 85.2), turned to 180 degrees
- moved U5 25.2 mm to (114.0, 87.9), turned to 90 degrees
- moved M0R1 19.5 mm to (208.2, 89.5), turned to 90 degrees
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Connections:
- A1 pad 14: M1-DIS -> M1-DIR
- A1 pad 15: M1-DIR -> M1-PWM
- A1 pad 16: M1-PWM -> M1-DIS
- A1 pad 40: Net-(A1-VBUS) -> VBUS
- A1 pad 5: PICO TX -> PICO-TX
- A1 pad 6: PICO RX -> PICO-RX
- C11 pad 1: Vdrive -> +3V3
- C12 pad 1: Vdrive -> GND
- C12 pad 2: GND -> Vdrive
- C13 pad 2: +3V3 -> Vdrive
- C2 pad 1: Vdrive -> GND
- C2 pad 2: GND -> +3V3
- C3 pad 1: Vdrive -> +3V3
- C4 pad 1: Vdrive -> +3V3
- C5 pad 1: +3V3 -> GND
- C5 pad 2: GND -> Vdrive
- C6 pad 1: +3V3 -> GND
- C6 pad 2: GND -> Vdrive
- C7 pad 1: +3V3 -> GND
- C7 pad 2: GND -> +3V3
- J1 pad 1: +12V -> GND
- J1 pad 2: GND -> +12V
- J1 pad 3: SERVO -> ADC
- J1 pad 4: ADC -> SERVO
- J2 pad 1: GND -> +12V
- J2 pad 2: Vdrive -> +5Vext
- J3 pad 1: +12V -> Net-(J3-Pin_1)
- J3 pad 2: +5V -> VBUS
- J3 pad 3: GND -> +5Vext
- J4 pad 1: Net-(J4-Pin_1) -> Net-(A1-USB_GND)
- J4 pad 2: Net-(A1-VBUS) -> Net-(A1-USB_DM)
- J4 pad 3: 5v -> Net-(A1-USB_DP)
- J5 pad 1: Net-(A1-USB_GND) -> GND
- J5 pad 2: Net-(A1-USB_DM) -> Vdrive
- J6 pad 3: 5v -> VBUS
- J6 pad 5: M0-B -> M0-A
- J6 pad 6: M0-A -> M0-B
- J7 pad 3: 5v -> VBUS
- J7 pad 5: M1-B -> M1-A
- J7 pad 6: M1-A -> M1-B
- J8 pad 3: 5v -> VBUS
- J9 pad 3: 5v -> VBUS
- M0R1 pad 1: GPIO16 -> GPIO17
- M0R2 pad 1: GPIO17 -> GPIO16
- M2R1 pad 1: GPIO22 -> GPIO21
- M2R2 pad 1: GPIO21 -> GPIO22
- U1 pad 1: M1-DIR -> M0-Enc-B
- U1 pad 2: +3V3 -> GND
- U1 pad 3: M1-SO -> M0-Enc-A
- U1 pad 4: Vdrive -> GPIO16
- U1 pad 5: M1-A -> +3V3
- U1 pad 6: GND -> GPIO17
- U2 pad 1: M3-DIR -> M2-Enc-B
- U2 pad 2: +3V3 -> GND
- U2 pad 3: PICO RX -> M2-Enc-A
- U2 pad 4: Vdrive -> GPIO22
- U2 pad 5: M3-A -> +3V3
- U2 pad 6: GND -> GPIO21
- U3 pad 1: M2-DIR -> M3-DIR
- U3 pad 11: M2-DIS -> M3-DIS
- U3 pad 12: M2-PWM -> M3-PWM
- U3 pad 3: M2-SO -> M3-SO
- U3 pad 5: M2-A -> M3-A
- U3 pad 7: M2-B -> M3-B
- U3 pad 8: M1-SO -> PICO-TX
- U4 pad 1: M0-DIR -> M1-DIR
- U4 pad 11: M0-DIS -> M1-DIS
- U4 pad 12: M0-PWM -> M1-PWM
- U4 pad 3: M0-SO -> M1-SO
- U4 pad 5: M0-A -> M1-A
- U4 pad 7: M0-B -> M1-B
- U4 pad 8: PICO TX -> M3-SO
- U5 pad 1: M3-Enc-B -> M1-Enc-B
- U5 pad 3: M3-Enc-A -> M1-Enc-A
- U5 pad 4: GPIO0 -> GPIO14
- U5 pad 6: GPIO1 -> GPIO15
- U6 pad 1: M0-Enc-B -> M3-Enc-B
- U6 pad 3: M0-Enc-A -> M3-Enc-A
- U6 pad 4: GPIO17 -> GPIO0
- U6 pad 6: GPIO16 -> GPIO1
- U7 pad 1: M2-Enc-B -> M2-DIR
- U7 pad 2: GND -> +3V3
- U7 pad 3: M2-Enc-A -> M2-SO
- U7 pad 4: GPIO21 -> Vdrive
- U7 pad 5: +3V3 -> M2-A
- U7 pad 6: GPIO22 -> GND
- U8 pad 1: M1-Enc-B -> M0-DIR
- U8 pad 2: GND -> +3V3
- U8 pad 3: M1-Enc-A -> M2-SO
- U8 pad 4: GPIO14 -> Vdrive
- U8 pad 5: +3V3 -> M0-A
- U8 pad 6: GPIO15 -> GND
Routing:
- net 5v: track 80.3 -> 0.00 mm, vias 1 -> 0
- net Vdrive: track 55.1 -> 0.00 mm, vias 9 -> 0
- net GND: track 26.3 -> 0.00 mm
- net M1-A: track 19.6 -> 0.00 mm, vias 2 -> 0
- net Net-(A1-VBUS): track 19.1 -> 0.00 mm
- net M1-PWM: track 18.1 -> 0.00 mm
- net (no net): track 16.4 -> 0.00 mm
- net M3-A: track 15.0 -> 0.00 mm
- net M1-B: track 12.2 -> 0.00 mm, vias 2 -> 0
- net M3-B: track 11.0 -> 0.00 mm
- net GPIO15: track 9.65 -> 0.00 mm
- net Net-(J4-Pin_1): track 7.48 -> 0.00 mm
- net GPIO17: track 7.03 -> 0.00 mm
- net GPIO21: track 6.80 -> 0.00 mm
- net GPIO16: track 6.63 -> 0.00 mm
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Other:
- board size 90.9 x 52.5 mm -> 90.9 x 70.1 mm

Commit message: trying again to get the PCB layout to work
Parts:
- J1, J4: footprint Connector_JST:JST_XH_S4B-XH-A_1x04_P2.50mm_Horizontal -> Connector_JST:JST_XH_B4B-XH-A_1x04_P2.50mm_Vertical
- J2: footprint Connector_JST:JST_XH_S3B-XH-A_1x03_P2.50mm_Horizontal -> Connector_JST:JST_XH_B3B-XH-A_1x03_P2.50mm_Vertical
- J6, J7, J8, J9: footprint Connector_JST:JST_XH_S6B-XH-A_1x06_P2.50mm_Horizontal -> Connector_JST:JST_XH_B6B-XH-A_1x06_P2.50mm_Vertical
- moved M0DB1 24.1 mm to (186.4, 85.3)
- moved M0R2 24.1 mm to (186.4, 88.8)
- moved M0DA1 24.0 mm to (184.2, 85.3)
- moved M0R1 24.0 mm to (184.2, 88.8)
- moved C2 22.4 mm to (183.7, 93.1), turned to 90 degrees
- moved C3 21.4 mm to (198.7, 88.1), turned to 90 degrees
- moved C13 18.2 mm to (198.7, 92.7), turned to 90 degrees
- moved J5 17.0 mm to (171.2, 89.0)
- moved U4 14.5 mm to (123.7, 89.4), turned to 90 degrees
- moved U8 13.7 mm to (192.6, 89.2), turned to 90 degrees
- moved C12 13.7 mm to (129.9, 92.9), turned to -90 degrees
- moved C8 13.1 mm to (118.1, 93.2), turned to 90 degrees
- moved C10 12.6 mm to (123.9, 60.2), turned to 90 degrees
- moved C6 12.4 mm to (112.5, 60.2), turned to 90 degrees
- moved J2 11.6 mm to (133.1, 98.6)
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Connections:
- net M3-SO renamed Net-(U3-SO)
- U4 pad 3: M1-SO -> Net-(U4-SO)
- U7 pad 3: M2-SO -> PICO-RX
- U7 pad 5: M2-A -> M2-B
- U7 pad 7: M2-B -> M2-A
- U7 pad 8: M1-SO -> Net-(U7-SI)
- U8 pad 3: M2-SO -> Net-(U7-SI)
- U8 pad 8: M1-SO -> Net-(U4-SO)
Routing:
- net VBUS: track 0.00 -> 206.9 mm, vias 0 -> 2
- net Vdrive: track 0.00 -> 143.2 mm, vias 0 -> 9
- net SCK: track 0.00 -> 114.4 mm, vias 0 -> 4
- net CSN: track 0.00 -> 109.1 mm, vias 0 -> 6
- net Net-(U4-SO): track 0.00 -> 86.3 mm, vias 0 -> 2
- net +5Vext: track 0.00 -> 78.7 mm, vias 0 -> 4
- net +3V3: track 0.00 -> 76.3 mm, vias 0 -> 17
- net M2-DIS: track 0.00 -> 56.9 mm, vias 0 -> 3
- net GPIO21: track 0.00 -> 50.5 mm, vias 0 -> 2
- net +12V: track 0.00 -> 46.2 mm
- net PICO-RX: track 0.00 -> 46.1 mm, vias 0 -> 3
- net GPIO22: track 0.00 -> 45.3 mm, vias 0 -> 2
- net GPIO15: track 0.00 -> 39.0 mm, vias 0 -> 2
- net ADC: track 0.00 -> 38.2 mm, vias 0 -> 1
- net SERVO: track 0.00 -> 37.1 mm
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Other:
- board size 90.9 x 70.1 mm -> 91.1 x 53 mm
